Commit message: Added planer move plugin. Also, corrected bot dimensions.

File: src/omnibot_description/urdf/omnibot.urdf (robot description, URDF)
Before this commit: robot omnibot, 1 links, 0 joints
Links:
- link base_link: geometry collision box size=3 2 0.4; visual box size=3 2 0.4

Commit message: Added Laser Plugin.
Also,

- Added robot state publisher and joint state publisher.

- Minor bugfixes.

File: src/omnibot_description/urdf/omnibot.urdf (robot description, URDF)
Before this commit: robot omnibot, 1 links, 0 joints
Links:
- added link hokuyo_link, mass 1e-5; collision box size=0.1 0.1 0.1; visual mesh filename=package://rrbot_description/meshes/hokuyo.dae
Joints:
- added joint hokuyo_joint: type fixed, parent base_link, child hokuyo_link, origin xyz=0 0 0.21 rpy=0 0 0, axis 0 1 0

Commit message: Corrected file name in laser visual and added the missing file.

File: src/omnibot_description/urdf/omnibot.urdf (robot description, URDF)
Before this commit: robot omnibot, 2 links, 1 joints
Links:
- link hokuyo_link: geometry collision box size=0.1 0.1 0.1; visual mesh filename=package://omnibot_description/meshes/hokuyo.dae
